File: AquaTank.sch (EAGLE design)
At the start: 1 part

Commit message: update
Parts:
- added SV1: (no value), con-lstb:MA20-2
Connections:
- new net 3V3: SV1.1, SV1.2, SV1.37, SV1.38
- new net GND: SV1.39, SV1.40
- new net PA0: SV1.5
- new net PA1: SV1.6
- new net PA10: SV1.31
- new net PA11: SV1.33
- new net PA12: SV1.34
- new net PA2: SV1.36
- new net PA3: SV1.35
- new net PA4: SV1.3
- new net PA9: SV1.32
- new net PB0: SV1.13
- new net PB1: SV1.16
- new net PB12: SV1.24
- new net PB13: SV1.23
- new net PB14: SV1.26
- new net PB15: SV1.25
- new net PB2: SV1.15
- new net PB5: SV1.18
- new net PC10: SV1.21
- new net PC11: SV1.22
- new net PC12: SV1.19
- new net PC2: SV1.7
- new net PC3: SV1.8
- new net PC7: SV1.27
- new net PC8: SV1.30
- new net PC9: SV1.29
- new net PD13: SV1.28
- new net PD2: SV1.20
- new net PD3: SV1.17
- new net PE0: SV1.4
- new net PE2: SV1.14
- new net PE3: SV1.11
- new net PE4: SV1.12
- new net PE5: SV1.9
- new net PE6: SV1.10
Other:
- note added: "DCF"
- note added: "Entree niveau osmolateur"
- note added: "PWM Eclairage"
- note added: "Pile"
